Commit message: 从gazebo world中读取 模型真值

File: gazebo_object_env/urdf/kinect.urdf.xacro (robot description, xacro)
@@ -42,5 +42,5 @@
   <!-- [2]  pose from camera to robot -->
   <xacro:property name="cam_px" value="0" />
-	<xacro:property name="cam_pz" value="0.2870" />
+	<xacro:property name="cam_pz" value="0.0" />
 	<xacro:property name="cam_or" value="0" />
 	<xacro:property name="cam_op" value="0" />
@@ -81,5 +81,5 @@
   	  </collision>
       <inertial>
-        <mass value="0.564" />
+        <mass value="0.000000000000001" />  <!-- 0.564 -->
         <origin xyz="0 0 0" />
         <inertia ixx="0.003881243" ixy="0.0" ixz="0.0"
